File: broadcast/hardware/circus_broadcast.kicad_pcb (KiCad board)
At the start: 2 copper layers, 37 parts, among them J301 M20-9990345, J302 M20-9990345, J402 M20-9990345, Q701 IRLML6244TRPBF, Q801 IRLML6244TRPBF, U201 LM317DCY, U301 LM317DCY, U302 LM317DCY, U401 C8051F850-C-GU, U501 LM317DCY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

Commit message: MOre lyaout
Parts:
- moved R304 127.2 mm to (21.7, 114.5), turned to 270 degrees
- moved R303 125.2 mm to (23.7, 114.5), turned to 270 degrees
- moved U501 123.7 mm to (51.5, 148.2), turned to 180 degrees
- moved R601 118.0 mm to (37.2, 144.1), turned to 180 degrees
- moved R501 114.3 mm to (45.2, 153.9)
- moved D701 103.5 mm to (56.5, 156.8), turned to 210 degrees
- moved R302 103.3 mm to (45.7, 115.5), turned to 270 degrees
- moved R301 103.0 mm to (45.7, 111.5), turned to 270 degrees
- moved J302 97.0 mm to (29.7, 121.5), turned to 90 degrees
- moved D702 92.2 mm to (60.4, 151.6), turned to 240 degrees
- moved R902 89.3 mm to (64.0, 134.0)
- moved J301 89.2 mm to (37.7, 121.5), turned to 90 degrees
- moved D703 88.1 mm to (59.1, 144.6), turned to 290 degrees
- moved D704 87.0 mm to (54.8, 140.2), turned to 330 degrees
- moved U301 86.4 mm to (37.7, 112.5)
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Routing:
- net Net-(J302-Pad1): track 0.00 -> 22.5 mm
- net Net-(R303-Pad1): track 0.00 -> 21.8 mm
- net +5V: track 0.00 -> 20.8 mm
- net CC1: track 0.00 -> 19.0 mm
- net CC2: track 0.00 -> 18.9 mm
- net GND: track 0.00 -> 15.3 mm
- net Net-(R301-Pad2): track 0.00 -> 12.8 mm
- net Net-(R601-Pad1): track 0.00 -> 12.3 mm
- net Net-(R501-Pad1): track 0.00 -> 12.2 mm
- net +3V3: track 0.00 -> 12.2 mm
- net Net-(R201-Pad2): track 0.00 -> 8.41 mm
- net Net-(D704-Pad1): track 0.00 -> 5.24 mm
- net Net-(D804-Pad1): track 0.00 -> 5.15 mm
- net Net-(D702-Pad1): track 0.00 -> 4.75 mm
- net Net-(D802-Pad1): track 0.00 -> 4.53 mm
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Other:
- board text added: "GND"
- board text added: "V+"
