File: broadcast/hardware/circus_broadcast.kicad_pcb (KiCad board)
At the start: 2 copper layers, 49 parts, among them J101 Keystone2238, J301 M20-9990345, J302 M20-9990345, J401 M20-9990445, J402 M20-9990345, Q701 IRLML6244TRPBF, Q801 IRLML6244TRPBF, T101 TestPoint, T401 TestPoint, T402 TestPoint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

Commit message: First passing layout
Parts:
- moved D901 71.1 mm to (39.9, 136.3), turned to 0 degrees
- moved R903 66.7 mm to (41.9, 139.7), turned to 90 degrees
- moved C601 62.2 mm to (35.6, 153.7), turned to 90 degrees
- moved U401 58.8 mm to (40.6, 144.8)
- moved J401 55.6 mm to (44.5, 138.4)
- moved U301 54.1 mm to (63.5, 160.0)
- moved U302 51.1 mm to (48.3, 160.0)
- moved C401 49.3 mm to (49.5, 144.1), turned to 270 degrees
- moved T101 47.5 mm to (53.3, 145.4)
- moved R304 47.1 mm to (45.7, 154.9)
- moved R301 46.1 mm to (61.0, 154.9)
- moved T402 44.9 mm to (53.3, 148.0)
- moved T401 44.6 mm to (53.3, 150.5)
- moved R303 43.9 mm to (40.6, 154.9)
- moved J301 42.6 mm to (55.9, 160.0), turned to 0 degrees
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Routing:
- net GND: track 15.3 -> 154.1 mm, vias 0 -> 7
- net +BATT: track 0.00 -> 75.1 mm, vias 0 -> 4
- net PWM1: track 0.00 -> 44.0 mm, vias 0 -> 4
- net LEDR: track 0.00 -> 39.9 mm, vias 0 -> 2
- net +3V3: track 12.2 -> 43.6 mm
- net MCU_RX: track 0.00 -> 28.9 mm, vias 0 -> 2
- net MCU_TX: track 0.00 -> 25.3 mm, vias 0 -> 2
- net PWM2: track 0.00 -> 17.1 mm, vias 0 -> 2
- net Net-(R401-Pad2): track 0.00 -> 12.6 mm, vias 0 -> 2
- net Net-(T402-Pad1): track 0.00 -> 12.2 mm, vias 0 -> 2
- net LEDG: track 0.00 -> 11.6 mm, vias 0 -> 2
- net Net-(T401-Pad1): track 0.00 -> 11.3 mm, vias 0 -> 2
- net Net-(R403-Pad1): track 0.00 -> 9.94 mm, vias 0 -> 2
- net Net-(J302-Pad1): track 22.5 -> 15.8 mm
- net +5V: track 20.8 -> 14.7 mm
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Other:
- board outline added: 77 x 28.5 mm

Commit message: tidy routing
Parts:
- moved T402 7.10 mm to (56.5, 141.6)
- moved T101 6.54 mm to (59.1, 148.6)
- moved R302 1.90 mm to (57.8, 154.9), turned to 180 degrees
- moved R401 1.42 mm to (52.1, 142.2)
- moved C201 0.90 mm to (70.5, 152.4), turned to 180 degrees
- turned R301 to 180 degrees
Routing:
- net GND: track 154.1 -> 189.2 mm, vias 7 -> 5
- net +5V: track 14.7 -> 32.4 mm, vias 0 -> 2
- net +3V3: track 43.6 -> 53.5 mm, vias 0 -> 2
- net Net-(J302-Pad1): track 15.8 -> 20.9 mm
- net Net-(T402-Pad1): track 12.2 -> 16.4 mm
- net Net-(T401-Pad1): track 11.3 -> 8.24 mm, vias 2 -> 0
- net +BATT: track 75.1 -> 78.2 mm
- net MCU_TX: track 25.3 -> 22.3 mm, vias 2 -> 1
- net MCU_RX: track 28.9 -> 26.3 mm, vias 2 -> 1
- net PWM1: track 44.0 -> 45.2 mm, vias 4 -> 2
- net Net-(R401-Pad2): track 12.6 -> 13.5 mm

Commit message: Final layout
Parts:
- moved R403 5.09 mm to (41.9, 142.5)
Routing:
- net +5V: track 32.4 -> 50.8 mm, vias 2 -> 4
- net +3V3: track 53.5 -> 69.1 mm, vias 2 -> 8
- net +BATT: track 78.2 -> 85.7 mm, vias 4 -> 5
- net Net-(R403-Pad1): track 9.94 -> 2.96 mm, vias 2 -> 0
- net Net-(J401-Pad2): track 2.81 -> 7.24 mm, vias 0 -> 1
- net LEDG: track 11.6 -> 14.8 mm
- net Net-(T402-Pad1): track 16.4 -> 18.8 mm
- net GND: track 189.2 -> 191.3 mm, vias 5 -> 4
- net Net-(R401-Pad2): track 13.5 -> 11.8 mm
- net PWM1: track 45.2 -> 43.7 mm
- net LEDR: track 39.7 -> 38.4 mm
- net MCU_RX: track 26.3 -> 27.3 mm
- added copper zone on B.Cu, net (none)
- added copper zone on F.Cu, net (none)
- added copper zone on B.Cu, net +3V3
- added copper zone on F.Cu, net +3V3
- added copper zone on B.Cu, net +BATT
- added copper zone on B.Cu, net GND
- added copper zone on F.Cu, net GND
- added copper zone on F.Cu, net Net-(J302-Pad1)
Other:
- board text added: "+9V"
- board text added: "1"
- board text added: "2"
- board text added: "Broadcast"
- board text added: "Circus"
- board text added: "G"
- board text added: "RevA Nov 2018"
- board text added: "Rx"
- board text added: "Tx"
